File: hardware/air-scales/air-scales.kicad_pcb (KiCad board)
At the start: 4 copper layers, 74 parts, among them J1 Connector, USB-TYPE-C-16P, J3 Conn_02x02_Odd_Even, J4 Conn_02x02_Odd_Even, J6 Conn_02x01, Q1 C458246, SW1 B3FS-1000, SW2 B3FS-1000, U1 BME280, U2 TPS62162DSG, U3 SMA6T28AY, U4 SMA6T15AY, U5 LM74610QDGKTQ1, U6 LM63625DQPWPRQ1, U7 TPS2553DRVR, U8 TPS2121RUXR, U9 ESP32-S3-WROOM-1U-N16R8

Commit message: need to redo a bunch of shit - lots of errors, totally fucked this all up
Parts:
- removed D6: GREEN, PCM_JLCPCB:D_0603
- removed R4: 100kΩ, PCM_JLCPCB:R_0603
- added C27: 100nF, PCM_JLCPCB:C_0603, F.Cu at (101.4, 63.8)
- added C28: 100nF, PCM_JLCPCB:C_0603, F.Cu at (101.4, 66.0)
- added C29: 100nF, PCM_JLCPCB:C_0603, F.Cu at (101.4, 68.3)
- added C30: 22uF, PCM_JLCPCB:C_1206, F.Cu at (106.1, 64.3)
- added D11: BLUE, PCM_JLCPCB:D_0603, F.Cu at (90.9, 87.4)
- added D12: ORANGE, PCM_JLCPCB:D_0603, F.Cu at (90.9, 83.6)
- added M1: MountingHole_3.2mm_M3_DIN965_Pad, MountingHole:MountingHole_3.2mm_M3_DIN965_Pad, F.Cu at (55.0, 45.0)
- added M2: MountingHole_3.2mm_M3_DIN965_Pad, MountingHole:MountingHole_3.2mm_M3_DIN965_Pad, F.Cu at (90.0, 45.0)
- added M3: MountingHole_3.2mm_M3_DIN965_Pad, MountingHole:MountingHole_3.2mm_M3_DIN965_Pad, F.Cu at (90.0, 130.0)
- added M4: MountingHole_3.2mm_M3_DIN965_Pad, MountingHole:MountingHole_3.2mm_M3_DIN965_Pad, F.Cu at (55.0, 130.0)
- added R21: 1.5kΩ, PCM_JLCPCB:R_0603, F.Cu at (86.3, 87.4)
- added R22: 1.5kΩ, PCM_JLCPCB:R_0603, F.Cu at (86.3, 83.6)
- D5: value Red -> RED
- D7: value YELLOW -> GREEN
- R16: value 10kΩ -> 5kΩ
- R19: value 470Ω -> 650Ω
- R20: value 1kΩ -> 1.5kΩ
- R3: value 1kΩ -> 10kΩ
- moved C12 34.3 mm to (68.8, 75.2)
- moved R11 31.9 mm to (86.2, 95.0), turned to 180 degrees
- moved U7 31.6 mm to (65.1, 79.8), turned to 90 degrees
- moved C14 29.8 mm to (71.5, 75.2)
- moved C13 29.8 mm to (66.2, 83.8), turned to 0 degrees
- moved J1 29.6 mm to (69.2, 130.0), turned to 0 degrees
- moved R7 28.1 mm to (72.2, 79.3), turned to -90 degrees
- moved R2 26.5 mm to (62.0, 124.1), turned to 180 degrees
- moved R8 23.4 mm to (70.5, 83.5), turned to 0 degrees
- moved R3 23.1 mm to (69.0, 79.3), turned to -90 degrees
- moved SW2 22.7 mm to (87.5, 101.5), turned to 0 degrees
- moved R15 22.5 mm to (77.8, 93.8), turned to 90 degrees
- moved C18 22.3 mm to (54.0, 121.7)
- moved C17 21.1 mm to (75.0, 73.5), turned to 90 degrees
- moved C22 21.1 mm to (74.8, 93.8)
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Connections:
- C12 pad 1: Net-(U7-IN) -> +5V ARB
- C13 pad 1: +5V USB -> +5V_SYS
- C14 pad 1: Net-(U7-EN) -> +5V ARB
- C17 pad 1: +5V_SYS -> +5V ARB
- C2 pad 2: Net-(U3-A) -> GND
- C26 pad 1: +5V USB -> VBUS
- C4 pad 1: Net-(U5-VCAPH) -> Net-(U5-VCAPL)
- C4 pad 2: Net-(U5-VCAPL) -> Net-(U5-VCAPH)
- C5 pad 1: Net-(Q1-D) -> +12VA
- C6 pad 1: Net-(Q1-D) -> +12VA
- C7 pad 1: Net-(Q1-D) -> +12VA
- D3 pad 2: Net-(U7-IN) -> VBUS
- D5 pad 2: Net-(U3-A) -> GND
- J1 pad A9B4: Net-(U7-IN) -> VBUS
- J1 pad B9A4: Net-(U7-IN) -> VBUS
- J3 pad 2: /U0TXD -> /U0RXD
- J3 pad 3: /U0RXD -> /U0TXD
- Q1 pad 5: Net-(Q1-D) -> +12VA
- R16 pad 1: +12V BATT -> +12VA
- R20 pad 1: +5V USB -> +5V VEHICLE
- R3 pad 1: +5V_SYS -> +5V ARB
- R3 pad 2: Net-(D6-Pad1) -> Net-(U7-EN)
- R7 pad 1: Net-(U7-IN) -> +5V ARB
- R7 pad 2: Net-(U7-EN) -> Net-(U7-~{FAULT})
- U3 pad 2: Net-(U3-A) -> GND
- U4 pad 1: Net-(U3-A) -> GND
- U5 pad 8: Net-(Q1-D) -> +12VA
- U6 pad 11: Net-(Q1-D) -> +12VA
- U6 pad 12: Net-(Q1-D) -> +12VA
- U6 pad 13: Net-(Q1-D) -> +12VA
- U7 pad 1: +5V USB -> +5V_SYS
- U7 pad 3: Net-(U7-EN) -> Net-(U7-~{FAULT})
- U7 pad 6: Net-(U7-IN) -> +5V ARB
- U8 pad 1: +5V_SYS -> +5V ARB
- U8 pad 1_1: +5V_SYS -> +5V ARB
- U8 pad 2: +5V USB -> VBUS
- U8 pad 2_1: unconnected-(U8-IN2__1-Pad2_1) -> VBUS
- U8 pad 3: Net-(U8-CP2) -> GND
- U8 pad 6: +5V VEHICLE -> GND
- U8 pad 7_1: unconnected-(U8-IN1__1-Pad7_1) -> +5V VEHICLE
- U8 pad 8: +5V_SYS -> +5V ARB
- U8 pad 8_1: +5V_SYS -> +5V ARB
- U8 pad 9: unconnected-(U8-ST-Pad9) -> GND
- U9 pad 16: /SDA -> unconnected-(U9-IO46-Pad16)
- U9 pad 17: /SCL -> unconnected-(U9-IO9-Pad17)
- U9 pad 21: /U0TXD -> /LED
- U9 pad 22: /U0RXD -> unconnected-(U9-IO14-Pad22)
- U9 pad 25: /PRESSURE_IN -> unconnected-(U9-IO48-Pad25)
- U9 pad 29: unconnected-(U9-IO36-Pad29) -> /PRESSURE_IN
- U9 pad 32: unconnected-(U9-IO39-Pad32) -> /SDA
- U9 pad 33: unconnected-(U9-IO40-Pad33) -> /SCL
- U9 pad 36: unconnected-(U9-RXD0-Pad36) -> /U0RXD
- U9 pad 37: unconnected-(U9-TXD0-Pad37) -> /U0TXD
- U9 pad 5: /LED -> unconnected-(U9-IO5-Pad5)
Routing:
- net GND: track 380.4 -> 223.0 mm, vias 134 -> 103
- net +12VA: track 0.00 -> 78.7 mm, vias 0 -> 2
- net +5V ARB: track 0.00 -> 62.8 mm
- net VBUS: track 0.00 -> 48.1 mm, vias 0 -> 2
- net Net-(Q1-D): track 32.9 -> 0.00 mm
- net +5V USB: track 27.8 -> 0.00 mm
- net +12V BATT: track 59.0 -> 31.4 mm, vias 2 -> 0
- net /BOOT: track 58.2 -> 31.7 mm
- net Net-(U3-A): track 18.2 -> 0.00 mm, vias 8 -> 0
- net +5V VEHICLE: track 15.8 -> 31.7 mm
- net /EN: track 31.0 -> 17.0 mm
- net /LED: track 38.8 -> 24.8 mm
- net Net-(U7-IN): track 11.1 -> 0.00 mm
- net +5V_SYS: track 52.5 -> 42.1 mm, vias 2 -> 0
- net /U0TXD: track 27.5 -> 37.4 mm, vias 0 -> 2
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- removed copper zone on In1.Cu, net GND
- removed copper zone on In2.Cu, net GND
Other:
- board outline added: 45 x 95 mm
- board text added: "12V"
- board text added: "3.3V"
- board text added: "5V"
- board text added: "Air Scales Part #"
- board text added: "JLCJLCJLCJLC"
- board text added: "V 0.02 by beaker 2025-11-21"
