File: hardware/AS 3/AS 3.kicad_sch (KiCad schematic)
At the start: 84 parts, among them J1 Conn_02x03_Odd_Even, J2 Conn_01x04, J3 USB_C_Receptacle_USB2.0_16P, Q1 PSMN5R2-60YL, SW1 SW_Push, SW2 SW_Push, U1 ESP32-S3-WROOM-1, U2 LM74610QDGKTQ1, U3 LMR604205SRAKRQ1, U4 TPS62901RPJR, U5 BME280, U6 TPS2121RUXR

Commit message: time for bom updates
Parts:
- J2: now not fitted; now left out of the parts list
- U3: footprint RAK0009A-MFG -> LMR60420:RAK0009A-MFG
Connections:
- net +3.3V: now also J2.4 (Pin_4); no longer J2.2 (Pin_2)
- net LED: now also U1.18 (IO10); no longer U1.28 (IO35)
- net PX3_PRESS: now also U1.17 (IO9); no longer U1.26 (IO45)
- net RXD0: now also J2.3 (Pin_3); no longer J2.4 (Pin_4)
- net TXD0: now also J2.2 (Pin_2); no longer J2.3 (Pin_3)
