File: hardware/AS 3/AS 3.kicad_sch (KiCad schematic)
At the start: 86 parts, among them J1 Conn_02x03_Odd_Even, J2 Conn_01x04, J3 USB_C_Receptacle_USB2.0_16P, Q1 IAUCN04S7N004, SW1 SW_Push, SW2 SW_Push, U1 ESP32-S3-WROOM-1, U2 LM74610QDGKTQ1, U3 LMR604205SRAKRQ1, U4 TPS62901RPJR, U5 BME280, U6 TPS2121RUXR

Commit message: order SMT025120460722-11369168A placed
Parts:
- added J4: Conn_01x02_Socket, Connector_PinHeader_1.00mm:PinHeader_1x02_P1.00mm_Vertical, symbol Connector:Conn_01x02_Socket
- added J5: Conn_01x03_Socket, Connector_PinHeader_1.00mm:PinHeader_1x03_P1.00mm_Vertical, symbol Connector:Conn_01x03_Socket
- C13: footprint Capacitor_SMD:CP_Elec_6.3x5.7 -> Capacitor_SMD:CP_Elec_6.3x7.7; LCSC C3274488 -> C28580967; Manufacturer KEMET -> Lelon; Mfr. Part # A768EB226M1HLAE048 -> VUP470M1HTR-0607; Voltage 50V -> (none)
- J3: FT Rotation Offset (none) -> 180
- L2: footprint Inductor_SMD:L_Chilisin_BMRF00101040 -> XGL6060-222MEC:IND_XGL6060_COC; LCSC C5562314 -> C3911671; Manufacturer Chilisin -> Coilcraft; Mfr. Part # AMRU001010402R2MA1 -> XGL6060-222MEC
- Q1: value IAUCN04S7N004 -> IAUC120N06S5L011
Connections:
- net +12V: now also J4.2 (Pin_2)
- net +5VMUX: now also J5.3 (Pin_3)
- net GND: now also J4.1 (Pin_1), J5.1 (Pin_1)
- net PX3_Signal: now also J5.2 (Pin_2)
