File: hardware/AS 3/_autosave-AS 3.kicad_pcb (KiCad board)
At the start: 4 copper layers, 45 x 65 mm, 84 parts, among them J1 Conn_02x03_Odd_Even, J2 Conn_01x04, J3 USB_C_Receptacle_USB2.0_16P, Q1 PSMN5R2-60YL, SW1 SW_Push, SW2 SW_Push, U1 ESP32-S3-WROOM-1, U2 LM74610QDGKTQ1, U3 LMR604205SRAKRQ1, U4 TPS62901RPJR, U5 BME280, U6 TPS2121RUXR

Commit message: time for bom updates
Parts:
- moved C5 15.5 mm to (74.8, 93.9)
- moved R9 0.79 mm to (63.2, 83.6), turned to 90 degrees
Routing:
- net GND: track 53.4 -> 54.1 mm

Commit message: ready to order the pcb
Parts:
- added C4: 10uF, Capacitor_SMD:C_0805_2012Metric, F.Cu at (60.3, 55.1)
- added R23: 15K, Resistor_SMD:R_0402_1005Metric, F.Cu at (63.3, 86.1)
- C1, C2, C21, C23, C5: footprint Capacitor_SMD:C_0402_1005Metric -> Capacitor_SMD:C_0603_1608Metric
- C11: value 4.7uF -> 10uF
- C15: value 10uF -> 100nF; footprint Capacitor_SMD:C_0805_2012Metric -> Capacitor_SMD:C_0603_1608Metric
- C17: value 18nF -> 22nF
- C19: value 22uF -> 10uF; footprint Capacitor_SMD:C_1206_3216Metric -> Capacitor_SMD:C_0805_2012Metric
- C24: value 10u -> 10uF
- C6: footprint Capacitor_SMD:C_0805_2012Metric -> Capacitor_SMD:C_0603_1608Metric
- C9: value 22uF -> 10uF
- D1, D4, D5, D6, D7: footprint LED_SMD:LED_0603_1608Metric -> LED_SMD:LED_0805_2012Metric
- L2: footprint Inductor_SMD:L_Chilisin_BMRF00101040 -> XGL6060-222MEC:IND_XGL6060_COC
- Q1: value PSMN5R2-60YL -> IAUC120N06S5L011; footprint Package_TO_SOT_SMD:LFPAK56 -> IAUC120N06S5L011:INF-PG-TDSON-8-33-V
- R10: value 86.6kΩ -> 82K
- R13: value 4,7K -> 4.7K
- R14: value 86.6kΩ -> 82K; footprint Resistor_SMD:R_0402_1005Metric -> Resistor_SMD:R_0603_1608Metric
- R16: value 16K -> 15K
- R17, R6: value 1k -> 1K
- R19: value 61.9K -> 47K
- moved C2 6.10 mm to (85.4, 105.3), turned to 90 degrees
- moved C10 5.52 mm to (81.2, 87.4)
- moved C22 5.48 mm to (81.2, 84.6)
- moved L2 3.87 mm to (74.4, 87.3)
- moved C5 2.78 mm to (77.6, 93.9), turned to 0 degrees
- moved Q1 2.20 mm to (69.8, 54.3)
- moved C19 1.23 mm to (60.3, 52.7)
- moved C3 1.15 mm to (85.4, 108.9)
- moved C1 0.95 mm to (86.1, 112.3)
- moved C24 0.92 mm to (85.7, 56.3), turned to 90 degrees
- moved R14 0.89 mm to (81.6, 61.7), turned to -90 degrees
- moved C23 0.82 mm to (83.7, 56.1), turned to 90 degrees
- moved C21 0.62 mm to (84.4, 112.3)
- moved R19 0.62 mm to (63.3, 87.3), turned to 180 degrees
- moved R15 0.53 mm to (81.4, 57.9), turned to -90 degrees
Connections:
- R19 pad 2: GND -> Net-(R19-Pad2)
Routing:
- net +5VBus: track 52.8 -> 48.4 mm, vias 9 -> 8
- net /SDA: track 60.5 -> 64.1 mm
- net Net-(U4-SW): track 13.3 -> 9.86 mm
- net +3.3V: track 28.3 -> 24.9 mm, vias 19 -> 18
- net GND: track 54.1 -> 52.4 mm, vias 105 -> 104
- net Net-(R19-Pad2): track 0.00 -> 1.26 mm
- net /PX3_PRESS: track 26.8 -> 27.9 mm
- net Net-(U2-VCAPL): track 8.48 -> 9.10 mm
- net /LED: track 21.1 -> 21.7 mm
- net +12V: vias 6 -> 10
Other:
- board text added: "-"
- board text removed: "AIR SCALES"
- board text removed: "v3"
