File: hardware/AS 3/AS 3.kicad_pcb (KiCad board)
At the start: 4 copper layers, 45 x 65 mm, 86 parts, among them J1 Conn_02x03_Odd_Even, J2 Conn_01x04, J3 USB_C_Receptacle_USB2.0_16P, Q1 IAUC120N06S5L011, SW1 SW_Push, SW2 SW_Push, U1 ESP32-S3-WROOM-1, U2 LM74610QDGKTQ1, U3 LMR604205SRAKRQ1, U4 TPS62901RPJR, U5 BME280, U6 TPS2121RUXR

Commit message: order SMT025120460722-11369168A placed
Parts:
- added FID1: Fiducial, Fiducial:Fiducial_1mm_Mask2mm, F.Cu at (103.0, 105.0)
- added FID2: Fiducial, Fiducial:Fiducial_1mm_Mask2mm, F.Cu at (103.0, 59.0)
- added FID3: Fiducial, Fiducial:Fiducial_1mm_Mask2mm, F.Cu at (44.0, 59.0)
- added FID4: Fiducial, Fiducial:Fiducial_1mm_Mask2mm, F.Cu at (44.0, 105.0)
- added J4: Conn_01x02_Socket, Connector_PinHeader_1.00mm:PinHeader_1x02_P1.00mm_Vertical, F.Cu at (52.2, 60.0)
- added J5: Conn_01x03_Socket, Connector_PinHeader_1.00mm:PinHeader_1x03_P1.00mm_Vertical, F.Cu at (52.9, 76.9)
- C13: footprint Capacitor_SMD:CP_Elec_6.3x5.7 -> Capacitor_SMD:CP_Elec_6.3x7.7
- moved R20 0.11 mm to (59.2, 93.0)
- moved R11 0.07 mm to (59.2, 87.7)
- moved R5 0.06 mm to (59.2, 82.5)
Routing:
- net /PX3_Signal: track 16.6 -> 20.4 mm
- net +12V: track 0.05 -> 1.07 mm, vias 10 -> 11
- net +5VMUX: track 24.0 -> 24.9 mm, vias 10 -> 11
- net GND: vias 104 -> 106
Other:
- board size 45 x 65 mm -> 71 x 75 mm
- board text added: "12V"
- board text added: "5V"
- board text added: "GND"
- board text added: "SIG"
- board text removed: "+"
- board text removed: "+5V-"
- board text removed: "-12V+"
- board text removed: "signal"
