File: hardware/AS 3/_autosave-AS 3.kicad_sch (KiCad schematic)
At the start: 86 parts, among them J1 Conn_02x03_Odd_Even, J2 Conn_01x04, J3 USB_C_Receptacle_USB2.0_16P, Q1 IAUCN04S7N004, SW1 SW_Push, SW2 SW_Push, U1 ESP32-S3-WROOM-1, U2 LM74610QDGKTQ1, U3 LMR604205SRAKRQ1, U4 TPS62901RPJR, U5 BME280, U6 TPS2121RUXR

Commit message: ready to order the pcb
Parts:
- L2: footprint Inductor_SMD:L_Chilisin_BMRF00101040 -> XGL6060-222MEC:IND_XGL6060_COC; LCSC C5562314 -> C3911671; Manufacturer Chilisin -> Coilcraft; Mfr. Part # AMRU001010402R2MA1 -> XGL6060-222MEC
- Q1: value IAUCN04S7N004 -> IAUC120N06S5L011
Changed lines of the file:
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@@
 			)
 		)
-		(property "Footprint" "Inductor_SMD:L_Chilisin_BMRF00101040"
+		(property "Footprint" "XGL6060-222MEC:IND_XGL6060_COC"
 			(at 328.93 95.25 0)
 			(effects
@@
 			)
 		)
-		(property "Datasheet" "https://www.lcsc.com/datasheet/C5562314.pdf"
+		(property "Datasheet" "https://www.coilcraft.com/getmedia/329fe97c-7311-4726-9bf3-37718f42b168/xgl6060.pdf"
 			(at 328.93 95.25 0)
 			(effects
@@
 			)
 		)
-		(property "Description" "FIXED IND 2.2uH 14A 6.8mΩ SMD,11.6x10.2mm"
+		(property "Description" "16A 2.2uH 4.9mΩ AEC-Q200 Magnetic Shielded Inductor ±20% SMD,6.7x6.5mm Power Inductors ROHS"
 			(at 328.93 95.25 0)
 			(effects
@@
 			)
 		)
-		(property "Manufacturer" "Chilisin"
+		(property "Manufacturer" " Coilcraft"
 			(at 328.93 95.25 0)
 			(effects
@@
 			)
 		)
-		(property "Mfr. Part #" "AMRU001010402R2MA1"
+		(property "Mfr. Part #" " XGL6060-222MEC"
 			(at 328.93 95.25 0)
 			(effects
@@
 			)
 		)
-		(property "LCSC" "C5562314"
+		(property "LCSC" " C3911671"
 			(at 328.93 95.25 0)
 			(effects
@@
 			)
 		)
+		(property "Voltage" ""
+			(at 328.93 95.25 0)
+			(effects
+				(font
+					(size 1.27 1.27)
+				)
+				(hide yes)
+			)
+		)
 		(pin "1"
 		)
@@
 			)
 		)
-		(property "Value" "IAUCN04S7N004"
+		(property "Value" "IAUC120N06S5L011"
 			(at 74.168 91.694 90)
 			(effects

Commit message: order SMT025120460722-11369168A placed
Parts:
- added FID1, FID2, FID3, FID4: Fiducial, Fiducial:Fiducial_1mm_Mask2mm, symbol Mechanical:Fiducial
- added J4: Conn_01x02_Socket, Connector_PinHeader_1.00mm:PinHeader_1x02_P1.00mm_Vertical, symbol Connector:Conn_01x02_Socket
- added J5: Conn_01x03_Socket, Connector_PinHeader_1.00mm:PinHeader_1x03_P1.00mm_Vertical, symbol Connector:Conn_01x03_Socket
- C13: footprint Capacitor_SMD:CP_Elec_6.3x5.7 -> Capacitor_SMD:CP_Elec_6.3x7.7; LCSC C3274488 -> C28580967; Manufacturer KEMET -> Lelon; Mfr. Part # A768EB226M1HLAE048 -> VUP470M1HTR-0607; Voltage 50V -> (none)
- J3: FT Rotation Offset (none) -> 180
Connections:
- net +12V: now also J4.2 (Pin_2)
- net +5VMUX: now also J5.3 (Pin_3)
- net GND: now also J4.1 (Pin_1), J5.1 (Pin_1)
- net PX3_Signal: now also J5.2 (Pin_2)
